Commit message: Added imu_link to urdf

File: orca_description/urdf/orca.urdf.xacro (robot description, xacro)
@@ -114,4 +114,36 @@
     <child link="enclosure"/>
   </joint>
+  <!-- IMU -->
+  <link name="imu_link">
+    <inertial>
+      <origin rpy="0 0 0" xyz="0 0 0"/>
+      <mass value="0"/>
+      <inertia
+        ixx="1.0" ixy="0.0" ixz="0.0"
+        iyy="1.0" iyz="0.0"
+        izz="1.0"/>
+    </inertial>
+    <visual>
+      <origin rpy="${PI/2} 0 0" xyz="0 0 0"/>
+      <geometry>
+        <box size="0.005 0.03 0.03"/>
+      </geometry>
+      <material name="red">
+        <color rgba="0.5 0 0 0.5"/>
+      </material>
+    </visual>
+    <collision>
+      <origin rpy="0 0 0" xyz="0 0 0"/>
+      <geometry>
+        <box size="0.005 0.03 0.03"/>
+      </geometry>
+    </collision>
+  </link>
+  <!-- Attach imu link to base link -->
+  <joint name="base_link_to_imu_link" type="fixed">
+    <origin rpy="0 0 0" xyz="0.025 0.10 0.06"/>
+    <parent link="base_link"/>
+    <child link="imu_link"/>
+  </joint>
   <!--
     Add Gazebo-specific elements to the base_link. See http://gazebosim.org/tutorials/?tut=ros_urdf for a list of allowed elements.
@@ -188,5 +220,5 @@
     The GazeboRosImuSensor (provided by ROS, wraps a Gazebo IMU sensor) simulates an IMU sensor such as the Phidgets 1044.
   -->
-  <gazebo reference="base_link">
+  <gazebo reference="imu_link">
     <gravity>true</gravity>
     <sensor name="imu_sensor" type="imu">
@@ -194,12 +226,12 @@
       <plugin filename="libgazebo_ros_imu_sensor.so" name="imu_plugin">
         <topicName>imu</topicName>
-        <bodyName>base_link</bodyName>
+        <bodyName>imu_link</bodyName>
         <updateRateHZ>100.0</updateRateHZ>
         <gaussianNoise>0.0</gaussianNoise> <!-- TODO -->
-        <xyzOffset>0 0 0</xyzOffset> <!-- TODO -->
-        <rpyOffset>0 0 0</rpyOffset> <!-- TODO -->
-        <frameName>base_link</frameName>
+        <xyzOffset>0 0 0</xyzOffset>
+        <rpyOffset>0 0 0</rpyOffset>
+        <frameName>imu_link</frameName>
       </plugin>
-      <pose>0 0 0 0 0 0</pose> <!-- TODO -->
+      <pose>0 0 0 0 0 0</pose>
     </sensor>
   </gazebo>

Commit message: Fixes after first underwater test

File: orca_description/urdf/orca.urdf.xacro (robot description, xacro)
@@ -1,3 +1,5 @@
 <?xml version="1.0"?>
+<!-- Coordinates are: x forward, y left, z up; rotation is: roll right, pitch forward, yaw left -->
+<!-- See http://www.ros.org/reps/rep-0103.html for details -->
 <robot name="orca" xmlns:xacro="http://ros.org/wiki/xacro">
   <!-- BlueROV2 specs -->
@@ -8,4 +10,7 @@
   <xacro:property name="WIDTH" value="0.338"/>
   <xacro:property name="HEIGHT" value="0.254"/>
+  <xacro:property name="THRUSTER_X" value="0.15"/>
+  <xacro:property name="THRUSTER_Y" value="0.1"/>
+  <xacro:property name="VERT_THRUSTER_Y" value="0.105"/>
   <!-- Physics properties -->
   <xacro:property name="FLUID_DENSITY" value="1000.0"/>
@@ -51,5 +56,5 @@
     <visual>
       <geometry>
-        <box size="${WIDTH} ${LENGTH} 0.01"/> <!--TODO eliminate visuals? -->
+        <box size="${LENGTH} ${WIDTH} 0.01"/>
       </geometry>
       <material name="gray">
@@ -59,5 +64,5 @@
     <collision>
       <geometry>
-        <box size="${WIDTH} ${LENGTH} 0.01"/> <!-- TODO set collision geometry to entire bounding box? -->
+        <box size="${LENGTH} ${WIDTH} 0.01"/>
       </geometry>
     </collision>
@@ -65,25 +70,25 @@
   <!-- Attach thrusters to the base_link -->
   <xacro:t200 name="front_right">
-    <origin xyz="0.1 0.15 0" rpy="0 ${PI/2} ${PI*3/4}"/>
+    <origin xyz="${THRUSTER_X} ${-THRUSTER_Y} 0" rpy="0 ${PI/2} ${PI*1/4}"/>
   </xacro:t200>
   <xacro:t200 name="front_left">
-    <origin xyz="-0.1 0.15 0" rpy="0 ${PI/2} ${PI*1/4}"/>
+    <origin xyz="${THRUSTER_X} ${THRUSTER_Y} 0" rpy="0 ${PI/2} ${-PI*1/4}"/>
   </xacro:t200>
   <xacro:t200 name="rear_right">
-    <origin xyz="0.1 -0.15 0" rpy="0 ${PI/2} ${PI*5/4}"/>
+    <origin xyz="${-THRUSTER_X} ${-THRUSTER_Y} 0" rpy="0 ${PI/2} ${PI*3/4}"/>
   </xacro:t200>
   <xacro:t200 name="rear_left">
-    <origin xyz="-0.1 -0.15 0" rpy="0 ${PI/2} ${PI*7/4}"/>
+    <origin xyz="${-THRUSTER_X} ${THRUSTER_Y} 0" rpy="0 ${PI/2} ${-PI*3/4}"/>
   </xacro:t200>
   <xacro:t200 name="vertical_right">
-    <origin xyz="0.105 0 0" rpy="0 0 0"/>
+    <origin xyz="0 ${-VERT_THRUSTER_Y} 0" rpy="0 0 0"/>
   </xacro:t200>
   <xacro:t200 name="vertical_left">
-    <origin xyz="-0.105 0 0" rpy="0 0 0"/>
+    <origin xyz="0 ${VERT_THRUSTER_Y} 0" rpy="0 0 0"/>
   </xacro:t200>
   <!-- Electronics enclosure -->
-  <link name="enclosure">
+  <link name="enclosure_link">
     <inertial>
-      <origin rpy="0 0 0" xyz="0 0 0"/>
+      <origin rpy="0 ${PI/2} 0" xyz="0 0 0"/>
       <mass value="${ENCLOSURE_MASS}"/>
       <inertia
@@ -93,5 +98,5 @@
     </inertial>
     <visual>
-      <origin rpy="${PI/2} 0 0" xyz="0 0 0"/>
+      <origin rpy="0 ${PI/2} 0" xyz="0 0 0"/>
       <geometry>
         <cylinder length="0.32" radius="0.055"/>
@@ -102,5 +107,5 @@
     </visual>
     <collision>
-      <origin rpy="${PI/2} 0 0" xyz="0 0 0"/>
+      <origin rpy="0 ${PI/2} 0" xyz="0 0 0"/>
       <geometry>
         <cylinder length="0.32" radius="0.055"/>
@@ -108,14 +113,14 @@
     </collision>
   </link>
-  <!-- Attach electronics enclosure to base link -->
-  <joint name="base_link_to_enclosure" type="fixed">
+  <!-- Attach enclosure link to base link -->
+  <joint name="base_link_to_enclosure_link" type="fixed">
     <origin rpy="0 0 0" xyz="0 0 0"/>
     <parent link="base_link"/>
-    <child link="enclosure"/>
+    <child link="enclosure_link"/>
   </joint>
   <!-- IMU -->
   <link name="imu_link">
     <inertial>
-      <origin rpy="0 0 0" xyz="0 0 0"/>
+      <origin rpy="${-PI/2} ${-PI/2} 0" xyz="0 0 0"/>
       <mass value="0"/>
       <inertia
@@ -125,16 +130,16 @@
     </inertial>
     <visual>
-      <origin rpy="${PI/2} 0 0" xyz="0 0 0"/>
-      <geometry>
-        <box size="0.005 0.03 0.03"/>
-      </geometry>
-      <material name="red">
-        <color rgba="0.5 0 0 0.5"/>
+      <origin rpy="${-PI/2} ${-PI/2} 0" xyz="0 0 0"/>
+      <geometry>
+        <box size="0.05 0.03 0.005"/>
+      </geometry>
+      <material name="green">
+        <color rgba="0 0.5 0 0.5"/>
       </material>
     </visual>
     <collision>
-      <origin rpy="0 0 0" xyz="0 0 0"/>
-      <geometry>
-        <box size="0.005 0.03 0.03"/>
+      <origin rpy="${-PI/2} ${-PI/2} 0" xyz="0 0 0"/>
+      <geometry>
+        <box size="0.05 0.03 0.005"/>
       </geometry>
     </collision>
@@ -142,7 +147,7 @@
   <!-- Attach imu link to base link -->
   <joint name="base_link_to_imu_link" type="fixed">
-    <origin rpy="0 0 0" xyz="0.025 0.10 0.06"/>
     <parent link="base_link"/>
     <child link="imu_link"/>
+    <origin rpy="0 0 0" xyz="0.1 -0.025 0.06"/>
   </joint>
   <!--
@@ -180,25 +185,25 @@
       <thruster name="front_right"> <!-- name attributes are ignored; the tag order must match the message array order -->
         <force>50</force> <!-- units are N, positive for ccw, negative for cw -->
-        <origin xyz="0.1 0.15 0" rpy="0 ${PI/2} ${PI*3/4}"/>
+        <origin xyz="${THRUSTER_X} ${-THRUSTER_Y} 0" rpy="0 ${PI/2} ${PI*1/4}"/>
       </thruster>
       <thruster name="front_left">
         <force>50</force>
-        <origin xyz="-0.1 0.15 0" rpy="0 ${PI/2} ${PI*1/4}"/>
+        <origin xyz="${THRUSTER_X} ${THRUSTER_Y} 0" rpy="0 ${PI/2} ${-PI*1/4}"/>
       </thruster>
       <thruster name="rear_right">
         <force>-50</force> <!-- cw -->
-        <origin xyz="0.1 -0.15 0" rpy="0 ${PI/2} ${PI*5/4}"/>
+        <origin xyz="${-THRUSTER_X} ${-THRUSTER_Y} 0" rpy="0 ${PI/2} ${PI*3/4}"/>
       </thruster>
       <thruster name="rear_left">
         <force>-50</force> <!-- cw -->
-        <origin xyz="-0.1 -0.15 0" rpy="0 ${PI/2} ${PI*7/4}"/>
+        <origin xyz="${-THRUSTER_X} ${THRUSTER_Y} 0" rpy="0 ${PI/2} ${-PI*3/4}"/>
       </thruster>
       <thruster name="vertical_right">
         <force>50</force>
-        <origin xyz="0.105 0 0" rpy="0 0 0"/>
+        <origin xyz="0 ${-VERT_THRUSTER_Y} 0" rpy="0 0 0"/>
       </thruster>
       <thruster name="vertical_left">
         <force>-50</force> <!-- cw -->
-        <origin xyz="-0.105 0 0" rpy="0 0 0"/>
+        <origin xyz="0 ${VERT_THRUSTER_Y} 0" rpy="0 0 0"/>
       </thruster>
     </plugin>
@@ -225,10 +230,10 @@
       <update_rate>100</update_rate>
       <plugin filename="libgazebo_ros_imu_sensor.so" name="imu_plugin">
-        <topicName>imu</topicName>
+        <topicName>/imu/data</topicName>
         <bodyName>imu_link</bodyName>
         <updateRateHZ>100.0</updateRateHZ>
-        <gaussianNoise>0.0</gaussianNoise> <!-- TODO -->
+        <gaussianNoise>0.0</gaussianNoise> <!-- TODO apply a noise model -->
         <xyzOffset>0 0 0</xyzOffset>
-        <rpyOffset>0 0 0</rpyOffset>
+        <rpyOffset>0 0 0</rpyOffset> <!-- TODO simulate a rotated imu -->
         <frameName>imu_link</frameName>
       </plugin>

Commit message: Throttle pid controllers if ROV is tilted

File: orca_description/urdf/orca.urdf.xacro (robot description, xacro)
@@ -13,4 +13,5 @@
   <xacro:property name="THRUSTER_Y" value="0.1"/>
   <xacro:property name="VERT_THRUSTER_Y" value="0.105"/>
+  <xacro:property name="BUOYANCY" value="0.1"/>
   <!-- Physics properties -->
   <xacro:property name="FLUID_DENSITY" value="1000.0"/>
@@ -48,5 +49,5 @@
     <inertial>
       <origin xyz="0 0 ${-HEIGHT / 3}"/> <!-- Center of mass is low -->
-      <mass value="${TOTAL_MASS - 6 * THRUSTER_MASS - ENCLOSURE_MASS}"/>
+      <mass value="${TOTAL_MASS - 6 * THRUSTER_MASS - ENCLOSURE_MASS - BUOYANCY}"/>
       <inertia
         ixx="1.0" ixy="0.0" ixz="0.0"
